File: PoE.kicad_sch (KiCad schematic)
At the start: 36 parts, among them J1001 8P8C_LED_Shielded_x2, J1002 8P8C_LED_Shielded_x2, U1001 7490220122, U1002 TCMT1107

Commit message: Added BOM, fixed routing mistakes
Parts:
- TP1001, TP1006: footprint SparkFun-Connector:TestPoint-1.0mm -> TestPoint:TestPoint_Pad_1.0x1.0mm
Changed lines of the file:
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@@
 			)
 		)
-		(property "Footprint" "SparkFun-Connector:TestPoint-1.0mm"
+		(property "Footprint" "TestPoint:TestPoint_Pad_1.0x1.0mm"
 			(at 271.78 76.2 0)
 			(effects
@@
 			)
 		)
-		(property "Footprint" "SparkFun-Connector:TestPoint-1.0mm"
+		(property "Footprint" "TestPoint:TestPoint_Pad_1.0x1.0mm"
 			(at 271.78 123.19 0)
 			(effects
