File: flyback.kicad_sch (KiCad schematic)
At the start: 48 parts, among them Q2 MMBT3906, Q2001 SI7898DP-T1-E3, U2001 TPS23751PWP, U2002 TCMT1107, U2003 TLV431ACDBZR

Commit message: Added BOM, fixed routing mistakes
Parts:
- C2003: footprint Capacitor_SMD:C_0805_2012Metric -> footprints:CAP_WCAP-ASLI_06p3X05p5_WRE
- C2009: footprint footprints:CAP_WCAP-ASLI_06p3X05p5_WRE -> Capacitor_SMD:C_0805_2012Metric
Connections:
- net at CR2003.2, T2001.2: now also Q2001.D
- net at D2.2 (A), T2001.5: no longer Q2001.D
Changed lines of the file:
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@@
 	)
 	(junction
+		(at 209.55 69.85)
+		(diameter 0)
+		(color 0 0 0 0)
+	)
+	(junction
 		(at 163.83 88.9)
 		(diameter 0)
@@
 		(color 0 0 0 0)
 	)
-	(junction
-		(at 209.55 83.82)
-		(diameter 0)
-		(color 0 0 0 0)
-	)
 	(no_connect
 		(at 97.79 93.98)
@@
 	(wire
 		(pts
-			(xy 209.55 83.82) (xy 214.63 83.82)
-		)
-		(stroke
-			(width 0)
-			(type default)
-		)
-	)
-	(wire
-		(pts
 			(xy 207.01 104.14) (xy 209.55 104.14)
 		)
@@
 	(wire
 		(pts
-			(xy 209.55 83.82) (xy 209.55 88.9)
-		)
-		(stroke
-			(width 0)
-			(type default)
-		)
-	)
-	(wire
-		(pts
 			(xy 97.79 119.38) (xy 100.33 119.38)
 		)
@@
 	(wire
 		(pts
+			(xy 209.55 69.85) (xy 209.55 88.9)
+		)
+		(stroke
+			(width 0)
+			(type default)
+		)
+	)
+	(wire
+		(pts
 			(xy 101.6 63.5) (xy 50.8 63.5)
 		)
@@
 	(wire
 		(pts
-			(xy 196.85 83.82) (xy 209.55 83.82)
+			(xy 196.85 83.82) (xy 214.63 83.82)
 		)
 		(stroke
@@
 			)
 		)
-		(property "Footprint" "footprints:CAP_WCAP-ASLI_06p3X05p5_WRE"
+		(property "Footprint" "Capacitor_SMD:C_0805_2012Metric"
 			(at 163.83 82.55 0)
 			(effects
@@
 			)
 		)
-		(property "Footprint" "Capacitor_SMD:C_0805_2012Metric"
+		(property "Footprint" "footprints:CAP_WCAP-ASLI_06p3X05p5_WRE"
 			(at 120.65 50.8 0)
 			(effects

Commit message: Prepping BOM
Parts:
- R2010: value 43.2 -> 49.9
- R2011: value 332 -> 470
- R2019: value 402 -> 470
- R2020: value 2k -> 2.2k
Changed lines of the file:
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@@
 			)
 		)
-		(property "Value" "43.2"
+		(property "Value" "49.9"
 			(at 143.51 95.25 90)
 			(effects
@@
 			)
 		)
-		(property "Value" "402"
+		(property "Value" "470"
 			(at 111.76 135.89 90)
 			(effects
@@
 			)
 		)
-		(property "Value" "2k"
+		(property "Value" "2.2k"
 			(at 111.76 146.05 90)
 			(effects
@@
 			)
 		)
-		(property "Value" "332"
+		(property "Value" "470"
 			(at 166.37 100.33 90)
 			(effects

Commit message: Fine tuning resistor values
Parts:
- R2008: value 10 -> 49.9
- R2011: value 470 -> 0
Changed lines of the file:
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@@
 			)
 		)
-		(property "Value" "10"
+		(property "Value" "49.9"
 			(at 179.07 85.09 90)
 			(effects
@@
 			)
 		)
-		(property "Value" "470"
+		(property "Value" "0"
 			(at 166.37 100.33 90)
 			(effects
